File: sensor_35mm.brd (EAGLE design)
At the start: 35.5 x 20.3 mm, 7 parts, among them J1 HEADER_SIDE_5POS, U1 HALL3-SIP, U2 HALL3-SIP, U3 HALL3-SIP

Commit message: just auto routed
Parts:
- removed J1: HEADER_SIDE_5POS, sc_usercreated:HEADER_SIDE_5POS
- added JP1: (no value), adafruit:1X03-CLEANBIG
- added JP2: M02PTH, SparkFun-Connectors:1X02
- moved C3 39.8 mm to (19.8, 6.60)
- moved U3 39.7 mm to (21.3, 4.55)
- moved U2 37.2 mm to (26.7, 5.36)
- moved C2 37.2 mm to (25.9, 7.87)
- moved C1 34.4 mm to (32.3, 7.11)
- moved U1 34.1 mm to (32.1, 4.55)
Connections:
- net +5V: now also JP2.1; no longer J1.4
- net GND: now also JP2.2; no longer J1.5
- net N$2: now also JP1.1; no longer J1.1
- net N$4: now also JP1.3; no longer J1.3
- net N$7: now also JP1.2; no longer J1.2
Routing:
- net N$2: track 21.7 -> 13.3 mm, vias 2 -> 0
- net N$4: track 19.0 -> 11.0 mm, vias 2 -> 0
- net N$7: track 15.0 -> 11.0 mm, vias 1 -> 0
- net GND: track 11.5 -> 7.67 mm, vias 1 -> 0
Other:
- board text added: "35"
- board text removed: "12t14p sensor board"
- board text removed: "30mm centers"
- board text removed: "59"
- board text removed: "85mm circle"
- board text removed: "etotheipiplusone.net"
- board text removed: "g5cba"
