File: sensor_35mm.sch (EAGLE design)
At the start: 7 parts, among them J1 HEADER_SIDE_5POS, U1 HALL3-SIP, U2 HALL3-SIP, U3 HALL3-SIP

Commit message: just auto routed
Parts:
- removed J1: HEADER_SIDE_5POS, sc_usercreated:HEADER_SIDE_5POS
- added JP1: (no value), adafruit:PINHD-1X3CB
- added JP2: M02PTH, SparkFun-Connectors:M02PTH
Connections:
- net +5V: now also JP2.1; no longer J1.4
- net GND: now also JP2.2; no longer J1.5
- net N$2: now also JP1.1; no longer J1.1
- net N$4: now also JP1.3; no longer J1.3
- net N$7: now also JP1.2; no longer J1.2
Changed lines of the file:
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@@
 <layer number="54" name="bGND_GNDA" color="1" fill="9" visible="no" active="no"/>
 <layer number="56" name="wert" color="7" fill="1" visible="no" active="no"/>
+<layer number="57" name="tCAD" color="7" fill="1" visible="no" active="no"/>
 <layer number="91" name="Nets" color="2" fill="1" visible="yes" active="yes"/>
 <layer number="92" name="Busses" color="1" fill="1" visible="yes" active="yes"/>
@@
 <layer number="97" name="Info" color="7" fill="1" visible="yes" active="yes"/>
 <layer number="98" name="Guide" color="6" fill="1" visible="yes" active="yes"/>
+<layer number="99" name="SpiceOrder" color="7" fill="1" visible="yes" active="yes"/>
 <layer number="100" name="Muster" color="7" fill="1" visible="no" active="no"/>
 <layer number="101" name="Patch_Top" color="12" fill="4" visible="no" active="yes"/>
@@
 <layer number="106" name="bPlate" color="7" fill="1" visible="no" active="yes"/>
 <layer number="107" name="Crop" color="7" fill="1" visible="no" active="yes"/>
+<layer number="108" name="fp8" color="7" fill="1" visible="no" active="yes"/>
+<layer number="109" name="fp9" color="7" fill="1" visible="no" active="yes"/>
+<layer number="110" name="fp0" color="7" fill="1" visible="no" active="yes"/>
+<layer number="111" name="LPC17xx" color="7" fill="1" visible="yes" active="yes"/>
+<layer number="112" name="tSilk" color="7" fill="1" visible="yes" active="yes"/>
+<layer number="113" name="IDFDebug" color="4" fill="1" visible="yes" active="yes"/>
 <layer number="116" name="Patch_BOT" color="9" fill="4" visible="no" active="yes"/>
 <layer number="121" name="_tsilk" color="7" fill="1" visible="no" active="yes"/>
 <layer number="122" name="_bsilk" color="7" fill="1" visible="no" active="yes"/>
+<layer number="123" name="tTestmark" color="7" fill="1" visible="no" active="yes"/>
+<layer number="124" name="bTestmark" color="7" fill="1" visible="no" active="yes"/>
 <layer number="125" name="_tNames" color="7" fill="1" visible="no" active="yes"/>
+<layer number="126" name="_bNames" color="7" fill="1" visible="yes" active="yes"/>
+<layer number="127" name="_tValues" color="7" fill="1" visible="yes" active="yes"/>
+<layer number="128" name="_bValues" color="7" fill="1" visible="yes" active="yes"/>
+<layer number="131" name="tAdjust" color="7" fill="1" visible="no" active="yes"/>
+<layer number="132" name="bAdjust" color="7" fill="1" visible="no" active="yes"/>
 <layer number="144" name="Drill_legend" color="7" fill="1" visible="no" active="yes"/>
+<layer number="150" name="Notes" color="7" fill="1" visible="no" active="yes"/>
 <layer number="151" name="HeatSink" color="7" fill="1" visible="no" active="yes"/>
+<layer number="152" name="_bDocu" color="7" fill="1" visible="yes" active="yes"/>
+<layer number="153" name="FabDoc1" color="6" fill="1" visible="no" active="no"/>
+<layer number="154" name="FabDoc2" color="2" fill="1" visible="no" active="no"/>
+<layer number="155" name="FabDoc3" color="7" fill="15" visible="no" active="no"/>
+<layer number="199" name="Contour" color="7" fill="1" visible="yes" active="yes"/>
 <layer number="200" name="200bmp" color="1" fill="10" visible="no" active="yes"/>
 <layer number="201" name="201bmp" color="2" fill="10" visible="no" active="yes"/>
@@
 <layer number="223" name="223bmp" color="24" fill="1" visible="no" active="no"/>
 <layer number="224" name="224bmp" color="25" fill="1" visible="no" active="no"/>
+<layer number="248" name="Housing" color="7" fill="1" visible="yes" active="yes"/>
+<layer number="249" name="Edge" color="7" fill="1" visible="yes" active="yes"/>
 <layer number="250" name="Descript" color="3" fill="1" visible="no" active="no"/>
 <layer number="251" name="SMDround" color="12" fill="11" visible="no" active="no"/>
@@
 <part name="P+4" library="supply1" deviceset="+5V" device=""/>
 <part name="GND4" library="supply1" deviceset="GND" device=""/>
-<part name="J1" library="sc_usercreated" deviceset="HEADER_SIDE_5POS" device=""/>
+<part name="JP1" library="adafruit" deviceset="PINHD-1X3" device="CB"/>
+<part name="JP2" library="SparkFun-Connectors" deviceset="M02" device="PTH"/>
 </parts>
 <sheets>
@@
 <instance part="GND2" gate="1" x="30.48" y="40.64"/>
 <instance part="GND3" gate="1" x="55.88" y="40.64"/>
-<instance part="P+4" gate="1" x="99.06" y="12.7"/>
-<instance part="GND4" gate="1" x="99.06" y="0" rot="MR0"/>
-<instance part="J1" gate="G$1" x="114.3" y="15.24" rot="R270"/>
+<instance part="P+4" gate="1" x="99.06" y="5.08"/>
+<instance part="GND4" gate="1" x="99.06" y="-7.62" rot="MR0"/>
+<instance part="JP1" gate="A" x="114.3" y="17.78"/>
+<instance part="JP2" gate="G$1" x="119.38" y="5.08" rot="R180"/>
 </instances>
 <busses>
@@
 </segment>
 <segment>
-<wire x1="99.06" y1="10.16" x2="99.06" y2="7.62" width="0.1524" layer="91"/>
-<wire x1="99.06" y1="7.62" x2="106.68" y2="7.62" width="0.1524" layer="91"/>
-<wire x1="106.68" y1="7.62" x2="106.68" y2="12.7" width="0.1524" layer="91"/>
-<wire x1="106.68" y1="12.7" x2="111.76" y2="12.7" width="0.1524" layer="91"/>
+<wire x1="99.06" y1="2.54" x2="99.06" y2="0" width="0.1524" layer="91"/>
+<wire x1="99.06" y1="0" x2="106.68" y2="0" width="0.1524" layer="91"/>
+<wire x1="106.68" y1="0" x2="106.68" y2="5.08" width="0.1524" layer="91"/>
+<wire x1="106.68" y1="5.08" x2="111.76" y2="5.08" width="0.1524" layer="91"/>
 <pinref part="P+4" gate="1" pin="+5V"/>
-<pinref part="J1" gate="G$1" pin="4"/>
+<pinref part="JP2" gate="G$1" pin="1"/>
 </segment>
 </net>
@@
 </segment>
 <segment>
-<wire x1="111.76" y1="10.16" x2="109.22" y2="10.16" width="0.1524" layer="91"/>
-<wire x1="109.22" y1="10.16" x2="109.22" y2="5.08" width="0.1524" layer="91"/>
-<wire x1="109.22" y1="5.08" x2="99.06" y2="5.08" width="0.1524" layer="91"/>
-<wire x1="99.06" y1="5.08" x2="99.06" y2="2.54" width="0.1524" layer="91"/>
-<pinref part="J1" gate="G$1" pin="5"/>
+<wire x1="111.76" y1="2.54" x2="109.22" y2="2.54" width="0.1524" layer="91"/>
+<wire x1="109.22" y1="2.54" x2="109.22" y2="-2.54" width="0.1524" layer="91"/>
+<wire x1="109.22" y1="-2.54" x2="99.06" y2="-2.54" width="0.1524" layer="91"/>
+<wire x1="99.06" y1="-2.54" x2="99.06" y2="-5.08" width="0.1524" layer="91"/>
 <pinref part="GND4" gate="1" pin="GND"/>
+<pinref part="JP2" gate="G$1" pin="2"/>
 </segment>
 </net>
@@
 <junction x="20.32" y="58.42"/>
 <pinref part="U1" gate="G$1" pin="OUT"/>
-<pinref part="J1" gate="G$1" pin="1"/>
+<pinref part="JP1" gate="A" pin="1"/>
 </segment>
 </net>
@@
 <junction x="71.12" y="58.42"/>
 <pinref part="U3" gate="G$1" pin="OUT"/>
-<pinref part="J1" gate="G$1" pin="3"/>
+<pinref part="JP1" gate="A" pin="3"/>
 </segment>
 </net>
@@
 <junction x="45.72" y="58.42"/>
 <pinref part="U2" gate="G$1" pin="OUT"/>
-<pinref part="J1" gate="G$1" pin="2"/>
-</segment>
-</net>
+<pinref part="JP1" gate="A" pin="2"/>
+</segment>
+</net>
